File: WirelessAction.kicad_pcb (KiCad board)
At the start: 2 copper layers, 43 x 30 mm, 13 parts, among them J1 Conn_01x08_Male, P1 RX, P2 TX, P3 SPARE, P4 -, P5 +, P6 -, P7 +, U1 WeMos_D1_mini

Commit message: Some minor changes
Parts:
- moved J1 2.30 mm to (108.6, 123.2)
Routing:
- net +3V3: track 39.6 -> 42.7 mm
- net /SCL: track 19.7 -> 22.1 mm
- net /SDA: track 10.8 -> 13.1 mm
- net /INT: track 24.5 -> 23.6 mm
- net GND: vias 2 -> 10
- added copper zone on B.Cu, net +3V3
- added copper zone on F.Cu, net +3V3
- added copper zone on F.Cu, net /INT
- added copper zone on F.Cu, net /SCL
- added copper zone on B.Cu, net /SDA
- added copper zone on F.Cu, net /SDA
- added copper zone on F.Cu, net /WARN
- added copper zone on F.Cu, net Net-(P1-Pad1)
- added copper zone on F.Cu, net Net-(P2-Pad1)
- added copper zone on F.Cu, net Net-(U1-Pad2)
- added copper zone on B.Cu, net VCC
- added copper zone on F.Cu, net VCC
